Commit message: update code

File: data/ewellix_lift_900mm.urdf.xacro (robot description, xacro)
@@ -9,5 +9,5 @@
         <origin xyz="0 0 0" rpy="0 0 0"/>
         <geometry>
-          <mesh filename="package://bmt_common_bringup/agv_descriptions/rbrobout/meshes/ewellix_lift_base_900mm.stl"/>
+          <mesh filename="package://dtc_test/meshes/ewellix_lift_base_900mm.stl"/>
         </geometry>
         <material name="grey">
@@ -18,5 +18,5 @@
         <origin xyz="-0.005 0 0.00235" rpy="0 0 0"/>
         <geometry>
-          <mesh filename="package://bmt_common_bringup/agv_descriptions/rbrobout/meshes/ewellix_lift_base_900mm.stl"/>
+          <mesh filename="package://dtc_test/meshes/ewellix_lift_base_900mm.stl"/>
         </geometry>
       </collision>
@@ -39,8 +39,8 @@
         <geometry>
           <xacro:if value="${cut_model}">
-            <mesh filename="package://bmt_common_bringup/agv_descriptions/rbrobout/meshes/ewellix_lift_top_900mm_cut.stl"/>
+            <mesh filename="package://dtc_test/meshes/ewellix_lift_top_900mm_cut.stl"/>
           </xacro:if>
           <xacro:unless value="${cut_model}">
-            <mesh filename="package://bmt_common_bringup/agv_descriptions/rbrobout/meshes/ewellix_lift_top_900mm.stl"/>
+            <mesh filename="package://dtc_test/meshes/ewellix_lift_top_900mm.stl"/>
           </xacro:unless>
         </geometry>
@@ -53,8 +53,8 @@
         <geometry>
           <xacro:if value="${cut_model}">
-            <mesh filename="package://bmt_common_bringup/agv_descriptions/rbrobout/meshes/ewellix_lift_top_900mm_cut.stl"/>
+            <mesh filename="package://dtc_test/meshes/ewellix_lift_top_900mm_cut.stl"/>
           </xacro:if>
           <xacro:unless value="${cut_model}">
-            <mesh filename="package://bmt_common_bringup/agv_descriptions/rbrobout/meshes/ewellix_lift_top_900mm.stl"/>
+            <mesh filename="package://dtc_test/meshes/ewellix_lift_top_900mm.stl"/>
           </xacro:unless>
         </geometry>

File: data/main.urdf.xacro (robot description, xacro)
@@ -46,7 +46,7 @@
     <xacro:arg name="safety_pos_margin" default="0.15" />
     <xacro:arg name="safety_k_position" default="20" />
-    <xacro:arg name="use_fake_hardware" default="false" />
+    <xacro:arg name="use_fake_hardware" default="true" />
     <xacro:arg name="fake_sensor_commands" default="false" />
-    <xacro:arg name="sim_gazebo" default="false" />
+    <xacro:arg name="sim_gazebo" default="true" />
     <xacro:arg name="sim_ignition" default="false" />
     <xacro:arg name="headless_mode" default="false" />
@@ -207,3 +207,10 @@
         <preserveFixedJoint>true</preserveFixedJoint>
     </gazebo>
+    <gazebo reference="world">
+    </gazebo>
+    <gazebo>
+      <plugin filename="libgazebo_ros2_control.so" name="gazebo_ros2_control">
+        <!--parameters>$(arg simulation_controllers)</parameters-->
+      </plugin>
+    </gazebo>
 </robot>
